File: A2VGA2/A2VGA.v2.1.kicad_pcb (KiCad board)
At the start: 2 copper layers, 65.5 x 79.8 mm, 66 parts, among them U1 CPB

Commit message: Add files via upload
Other:
- board text added: "A2VGA.v2.0 Board design by Ralle Palaveev, (c) 2026 www.apple2.co.uk Firmware by Oliver Schmidt, (c) 2026 https://a2retro.de/ Based on work by: AppleII-VGA, Mark Aikens (c) 2021-2023 Analog Firmware, David Kuder (c) 2022-2023"
- board text removed: "A2VGA.v2.1 Board design by R.Palaveev (c) 2026 www.apple2.co.uk Based on work by: AppleII-VGA, Mark Aikens (c) 2021-2023 Analog Firmware, David Kuder (c) 2022-2023"
Changed lines of the file:
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@@
 		)
 	)
-	(gr_text "A2VGA.v2.1\nBoard design by R.Palaveev (c) 2026\nwww.apple2.co.uk\n\nBased on work by:\nAppleII-VGA, Mark Aikens (c) 2021-2023\nAnalog Firmware, David Kuder (c) 2022-2023"
+	(gr_text "A2VGA.v2.0\nBoard design by Ralle Palaveev, (c) 2026\nwww.apple2.co.uk\nFirmware by Oliver Schmidt, (c) 2026\nhttps://a2retro.de/\nBased on work by:\nAppleII-VGA, Mark Aikens (c) 2021-2023\nAnalog Firmware, David Kuder (c) 2022-2023"
 		(at 148.0312 112.5982 0)
 		(layer "B.SilkS")
 		(effects
 			(font
-				(size 1 1)
+				(size 0.8 0.9)
 				(thickness 0.2)
 			)

Commit message: Add files via upload
Connections:
- ? pad 1: ~{IOSel} -> (no net)
- ? pad 20: ~{IOStr} -> (no net)
- U1 pad 48: ~{IOSel} -> (no net)
- U1 pad 49: ~{IOStr} -> (no net)
Routing:
- net ~{IOSel}: track 67.4 -> 0.00 mm, vias 1 -> 0
- net ~{IOStr}: track 30.8 -> 0.00 mm, vias 2 -> 0
Changed lines of the file:
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@@
 	(net 48 "VBUS")
 	(net 49 "SYNC")
-	(net 50 "~{IOSel}")
-	(net 51 "~{IOStr}")
 	(footprint ""
 		(layer "F.Cu")
@@
 			(size 1.524 6.35)
 			(layers "F.Cu" "F.Mask")
-			(net 50 "~{IOSel}")
 		)
 	)
@@
 			(layers "*.Cu" "*.Mask")
 			(remove_unused_layers no)
-			(net 50 "~{IOSel}")
 		)
 		(pad "49" thru_hole oval
@@
 			(layers "*.Cu" "*.Mask")
 			(remove_unused_layers no)
-			(net 51 "~{IOStr}")
 		)
 		(pad "50" thru_hole oval
@@
 			(size 1.524 6.35)
 			(layers "F.Cu" "F.Mask")
-			(net 51 "~{IOStr}")
 		)
 	)
@@
 		(net 49)
 	)
-	(segment
-		(start 112.4458 111.76)
-		(end 112.4458 127.762)
-		(width 0.2)
-		(layer "F.Cu")
-		(net 50)
-	)
-	(segment
-		(start 112.4458 127.762)
-		(end 114.3 129.6162)
-		(width 0.2)
-		(layer "F.Cu")
-		(net 50)
-	)
-	(segment
-		(start 114.3 129.6162)
-		(end 114.3 135.519807)
-		(width 0.2)
-		(layer "F.Cu")
-		(net 50)
-	)
-	(segment
-		(start 113.6142 110.5916)
-		(end 112.4458 111.76)
-		(width 0.2)
-		(layer "F.Cu")
-		(net 50)
-	)
-	(via
-		(at 113.6142 110.5916)
-		(size 0.8)
-		(drill 0.4)
-		(layers "F.Cu" "B.Cu")
-		(net 50)
-	)
-	(segment
-		(start 116.0272 110.617)
-		(end 153.0604 110.617)
-		(width 0.2)
-		(layer "B.Cu")
-		(net 50)
-	)
-	(segment
-		(start 113.6142 110.5916)
-		(end 116.0018 110.5916)
-		(width 0.2)
-		(layer "B.Cu")
-		(net 50)
-	)
-	(segment
-		(start 153.0604 110.617)
-		(end 154.3304 111.887)
-		(width 0.2)
-		(layer "B.Cu")
-		(net 50)
-	)
-	(segment
-		(start 116.0018 110.5916)
-		(end 116.0272 110.617)
-		(width 0.2)
-		(layer "B.Cu")
-		(net 50)
-	)
-	(segment
-		(start 158.5722 115.6716)
-		(end 158.1404 115.2398)
-		(width 0.2)
-		(layer "F.Cu")
-		(net 51)
-	)
-	(segment
-		(start 164.2872 115.6716)
-		(end 164.2872 129.1844)
-		(width 0.2)
-		(layer "F.Cu")
-		(net 51)
-	)
-	(segment
-		(start 164.2872 129.1844)
-		(end 162.56 130.9116)
-		(width 0.2)
-		(layer "F.Cu")
-		(net 51)
-	)
-	(segment
-		(start 158.1404 115.2398)
-		(end 158.1404 113.792)
-		(width 0.2)
-		(layer "F.Cu")
-		(net 51)
-	)
-	(segment
-		(start 160.528 115.6716)
-		(end 158.5722 115.6716)
-		(width 0.2)
-		(layer "F.Cu")
-		(net 51)
-	)
-	(segment
-		(start 156.8704 112.522)
-		(end 156.8704 111.887)
-		(width 0.2)
-		(layer "F.Cu")
-		(net 51)
-	)
-	(segment
-		(start 158.1404 113.792)
-		(end 156.8704 112.522)
-		(width 0.2)
-		(layer "F.Cu")
-		(net 51)
-	)
-	(segment
-		(start 162.56 130.9116)
-		(end 162.56 135.519807)
-		(width 0.2)
-		(layer "F.Cu")
-		(net 51)
-	)
-	(via
-		(at 160.528 115.6716)
-		(size 0.8)
-		(drill 0.4)
-		(layers "F.Cu" "B.Cu")
-		(net 51)
-	)
-	(via
-		(at 164.2872 115.6716)
-		(size 0.8)
-		(drill 0.4)
-		(layers "F.Cu" "B.Cu")
-		(net 51)
-	)
-	(segment
-		(start 160.528 115.6716)
-		(end 164.2872 115.6716)
-		(width 0.2)
-		(layer "B.Cu")
-		(net 51)
-	)
 	(zone
