File: A2VGA2/A2VGA.v2.1.kicad_pcb (KiCad board)
At the start: 2 copper layers, 65.5 x 79.8 mm, 66 parts, among them U1 CPB

Commit message: Add files via upload
Routing:
- net GND: vias 35 -> 36
Changed lines of the file:
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@@
+	)
+	(via
+		(at 144.1704 111.3536)
+		(size 0.6)
+		(drill 0.3)
+		(layers "F.Cu" "B.Cu")
+		(free yes)
+		(net 1)
 	)
 	(via
