File: A2VGA2/A2VGA.v2.0.kicad_pcb (KiCad board)
At the start: 2 copper layers, 92.8 x 46.8 mm, 68 parts, among them U1 CPB

Commit message: Add files via upload
Routing:
- net GND: vias 30 -> 31
Changed lines of the file:
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@@
+	)
+	(via
+		(at 144.1958 111.2012)
+		(size 0.8)
+		(drill 0.4)
+		(layers "F.Cu" "B.Cu")
+		(free yes)
+		(net 1)
 	)
 	(via
