File: A2VGA2/HW/A2VGA.v2.2.kicad_pcb (KiCad board)
At the start: 2 copper layers, 65.5 x 79.8 mm, 66 parts, among them U1 CPB

Commit message: Add files via upload
Parts:
- moved H3 39.0 mm to (125.0, 71.4), turned to 90 degrees
Routing:
- net HS_out: track 86.2 -> 21.4 mm
- net VS_out: track 76.7 -> 23.9 mm
- net R_out: track 29.9 -> 62.8 mm
- net B_out: track 52.5 -> 38.3 mm
- net G_out: track 41.6 -> 50.9 mm
- net GND: track 4.95 -> 12.0 mm, vias 36 -> 30
Other:
- outline, holes or cut-outs redrawn
- board text added: "A2VGA.v2.2 (c) 2026 by Ralle Palaveev, https://apple2.co.uk/"
- board text removed: "A2VGA.v2.1 (c) 2026 by Ralle Palaveev, https://apple2.co.uk/"

Commit message: Add files via upload
Parts:
- D1: value D_T-1_P5.08mm_Horizontal -> 1N5819
- moved G*** 12.8 mm to (170.0, 114.8)
Connections:
- U1 pad 37: (no net) -> VSYS
Routing:
- net VSYS: track 5.98 -> 12.3 mm
Other:
- board text added: "A2VGA.v2.2"
- board text added: "Keyboard this way"
- board text removed: "A2VGA.v2.1"
