File: A2VGA2/HW/A2VGA.v2.2.kicad_pcb (KiCad board)
At the start: 2 copper layers, 65.5 x 79.8 mm, 66 parts, among them U1 CPB

Commit message: Add files via upload
Routing:
- net GND: track 12.0 -> 14.1 mm
Changed lines of the file:
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@@
 	)
 	(segment
-		(start 126.961869 79.3816)
-		(end 125.816869 80.5266)
+		(start 126.167069 81.7118)
+		(end 124.981869 80.5266)
+		(width 0.4)
+		(layer "F.Cu")
+		(net 1)
+	)
+	(segment
+		(start 126.961869 81.368931)
+		(end 126.619 81.7118)
 		(width 0.4)
 		(layer "F.Cu")
@@
 	)
 	(segment
-		(start 125.816869 80.5266)
-		(end 124.981869 80.5266)
+		(start 126.619 81.7118)
+		(end 126.167069 81.7118)
 		(width 0.4)
 		(layer "F.Cu")
+		(net 1)
+	)
+	(segment
+		(start 126.961869 79.3816)
+		(end 126.961869 81.368931)
+		(width 0.4)
+		(layer "F.Cu")

Commit message: Add files via upload
Parts:
- added C2: 100n, Capacitor_THT:C_Disc_D5.0mm_W2.5mm_P5.00mm, F.Cu at (120.3, 97.1)
- moved C1 2.96 mm to (120.3, 94.0)
Connections:
- U1 pad 30: (no net) -> RUN
Routing:
- net RUN: track 0.00 -> 17.3 mm
- net 5V: track 100.9 -> 102.4 mm
- net GND: vias 30 -> 34

Commit message: Add files via upload
Parts:
- added R12: 1k, Resistor_THT:R_Axial_DIN0204_L3.6mm_D1.6mm_P5.08mm_Horizontal, F.Cu at (130.1, 95.8)
Routing:
- net 3.3V: track 0.00 -> 12.4 mm
- net GND: vias 34 -> 36

Commit message: Add files via upload
Parts:
- removed C2: 100n, Capacitor_THT:C_Disc_D5.0mm_W2.5mm_P5.00mm
- moved C1 2.40 mm to (119.4, 96.2)
- moved R12 0.05 mm to (130.2, 95.8)
Routing:
- net RUN: track 17.3 -> 11.5 mm
- net 5V: track 102.4 -> 101.6 mm
- net GND: vias 36 -> 37
