File: A2VGA2/HW/A2VGA.v2.0.kicad_pcb (KiCad board)
At the start: 2 copper layers, 92.8 x 46.8 mm, 68 parts, among them U1 CPB

Commit message: Add files via upload
Routing:
- net GND: track 4.95 -> 12.0 mm
Changed lines of the file:
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@@
 		(tags "Resistor Axial_DIN0204 series Axial Horizontal pin pitch 5.08mm 0.167W length 3.6mm diameter 1.6mm")
 		(property "Reference" "R4"
-			(at 2.6162 -0.0254 90)
+			(at -1.524 -0.0508 180)
 			(layer "F.SilkS")
 			(effects
@@
 		(property "Value" "510"
 			(at 2.54 0 90)
-			(layer "F.Fab")
+			(layer "F.SilkS")
 			(effects
 				(font
@@
 		(tags "Resistor Axial_DIN0204 series Axial Horizontal pin pitch 5.08mm 0.167W length 3.6mm diameter 1.6mm")
 		(property "Reference" "R3"
-			(at 2.5654 0 90)
+			(at -1.5494 -0.0508 180)
 			(layer "F.SilkS")
 			(effects
@@
 		(property "Value" "2k"
 			(at 2.54 0 90)
-			(layer "F.Fab")
+			(layer "F.SilkS")
 			(effects
 				(font
@@
 		(tags "Resistor Axial_DIN0204 series Axial Horizontal pin pitch 5.08mm 0.167W length 3.6mm diameter 1.6mm")
 		(property "Reference" "R9"
-			(at 2.5146 0.0762 90)
+			(at -1.524 0 180)
 			(layer "F.SilkS")
 			(effects
@@
 		)
 		(property "Value" "2k"
-			(at 2.54 0 90)
-			(layer "F.Fab")
+			(at 2.54 0 -90)
+			(layer "F.SilkS")
 			(effects
 				(font
@@
 		(tags "Resistor Axial_DIN0204 series Axial Horizontal pin pitch 5.08mm 0.167W length 3.6mm diameter 1.6mm")
 		(property "Reference" "R2"
-			(at 2.5146 0 90)
+			(at -1.5748 -0.0254 180)
 			(layer "F.SilkS")
 			(effects
@@
 		(property "Value" "1k"
 			(at 2.54 0 90)
-			(layer "F.Fab")
+			(layer "F.SilkS")
 			(effects
 				(font
@@
 		(tags "Resistor Axial_DIN0204 series Axial Horizontal pin pitch 5.08mm 0.167W length 3.6mm diameter 1.6mm")
 		(property "Reference" "R1"
-			(at 2.7686 0 90)
+			(at -1.5494 -0.0508 180)
 			(layer "F.SilkS")
 			(effects
@@
 		(property "Value" "510"
 			(at 2.54 0 90)
-			(layer "F.Fab")
+			(layer "F.SilkS")
 			(effects
 				(font
@@
 		(tags "Resistor Axial_DIN0204 series Axial Horizontal pin pitch 5.08mm 0.167W length 3.6mm diameter 1.6mm")
 		(property "Reference" "R7"
-			(at 2.5654 0.0254 90)
+			(at -1.5494 -0.0254 180)
 			(layer "F.SilkS")
 			(effects
@@
 		(property "Value" "510"
 			(at 2.54 0 90)
-			(layer "F.Fab")
+			(layer "F.SilkS")
 			(effects
 				(font
@@
 		(tags "Resistor Axial_DIN0204 series Axial Horizontal pin pitch 5.08mm 0.167W length 3.6mm diameter 1.6mm")
 		(property "Reference" "R11"
-			(at 2.667 0 90)
+			(at -1.5494 0.0508 180)
 			(layer "F.SilkS")
 			(effects
@@
 		(property "Value" "47"
 			(at 2.54 0 90)
-			(layer "F.Fab")
+			(layer "F.SilkS")
 			(effects
 				(font
@@
 		(tags "Resistor Axial_DIN0204 series Axial Horizontal pin pitch 5.08mm 0.167W length 3.6mm diameter 1.6mm")
 		(property "Reference" "R10"
-			(at 2.5654 0.0254 90)
+			(at -1.5494 -0.0508 180)
 			(layer "F.SilkS")
 			(effects
@@
 		(property "Value" "47"
 			(at 2.54 0 90)
-			(layer "F.Fab")
+			(layer "F.SilkS")
 			(effects
 				(font
@@
 		(tags "Resistor Axial_DIN0204 series Axial Horizontal pin pitch 5.08mm 0.167W length 3.6mm diameter 1.6mm")
 		(property "Reference" "R6"
-			(at 2.5654 0 90)
+			(at -1.5748 0.0254 180)
 			(layer "F.SilkS")
 			(effects
@@
 		(property "Value" "2k"
 			(at 2.54 0 90)
-			(layer "F.Fab")
+			(layer "F.SilkS")
 			(effects
 				(font
@@
 		(tags "Resistor Axial_DIN0204 series Axial Horizontal pin pitch 5.08mm 0.167W length 3.6mm diameter 1.6mm")
 		(property "Reference" "R8"
-			(at 2.4638 0.0508 90)
+			(at -1.524 0.0254 180)
 			(layer "F.SilkS")
 			(effects
@@
 		(property "Value" "1k"
 			(at 2.54 0 90)
-			(layer "F.Fab")
+			(layer "F.SilkS")
 			(effects
 				(font
@@
 		(tags "Resistor Axial_DIN0204 series Axial Horizontal pin pitch 5.08mm 0.167W length 3.6mm diameter 1.6mm")
 		(property "Reference" "R5"
-			(at 2.5146 0 90)
+			(at -1.5494 0.0508 180)
 			(layer "F.SilkS")
 			(effects
@@
 		(property "Value" "1k"
 			(at 2.54 0 90)
-			(layer "F.Fab")
+			(layer "F.SilkS")
 			(effects
 				(font
@@
 		(net 0)
 	)
+	(segment
+		(start 193.478 115.7426)
+		(end 192.643 115.7426)
+		(width 0.4)
+		(layer "F.Cu")
+		(net 1)
+	)
+	(segment
+		(start 193.478 106.5826)
+		(end 193.478 111.1626)
+		(width 0.4)
+		(layer "F.Cu")
+		(net 1)
+	)
+	(segment
+		(start 192.643 115.7426)
+		(end 191.498 116.8876)
+		(width 0.4)
+		(layer "F.Cu")
+		(net 1)
+	)
 	(via

Commit message: Add files via upload
Parts:
- added C2: 100n, Capacitor_THT:C_Disc_D5.0mm_W2.5mm_P5.00mm, F.Cu at (120.3, 97.1)
- moved C1 2.93 mm to (120.2, 94.0)
Connections:
- U1 pad 30: (no net) -> RUN
- U1 pad 37: (no net) -> VSYS
Routing:
- net RUN: track 0.00 -> 17.3 mm
- net VSYS: track 5.98 -> 12.4 mm
- net 5V: track 101.0 -> 102.8 mm

Commit message: Add files via upload
Parts:
- added R12: 1k, Resistor_THT:R_Axial_DIN0204_L3.6mm_D1.6mm_P5.08mm_Horizontal, F.Cu at (130.1, 95.8)
Routing:
- net 3.3V: track 0.00 -> 12.4 mm
- net GND: vias 31 -> 35
