File: A2VGA2/HW/A2VGA.v2.1.kicad_pcb (KiCad board)
At the start: 2 copper layers, 65.5 x 79.8 mm, 66 parts, among them U1 CPB

Commit message: Add files via upload
Routing:
- net GND: track 4.95 -> 12.0 mm
Changed lines of the file:
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@@
 		(net 0)
+	)
+	(segment
+		(start 163.1114 70.4628)
+		(end 162.505 71.0692)
+		(width 0.4)
+		(layer "F.Cu")
+		(net 1)
+	)
+	(segment
+		(start 161.1314 78.4778)
+		(end 161.1314 80.7678)
+		(width 0.4)
+		(layer "F.Cu")
+		(net 1)
+	)
+	(segment
+		(start 162.505 71.0692)
+		(end 161.67 71.0692)
+		(width 0.4)
+		(layer "F.Cu")
+		(net 1)
+	)
+	(segment
+		(start 161.1314 78.4778)
+		(end 161.1314 76.1878)
+		(width 0.4)
+		(layer "F.Cu")
+		(net 1)
+	)
+	(segment
+		(start 161.67 71.0692)
+		(end 161.1314 71.6078)
+		(width 0.4)
+		(layer "F.Cu")
+		(net 1)
 	)
 	(via

Commit message: Add files via upload
Parts:
- added C2: 100n, Capacitor_THT:C_Disc_D5.0mm_W2.5mm_P5.00mm, F.Cu at (120.3, 97.1)
- moved C1 2.93 mm to (120.3, 94.0)
Connections:
- U1 pad 30: (no net) -> RUN
- U1 pad 37: (no net) -> VSYS
Routing:
- net RUN: track 0.00 -> 17.3 mm
- net VSYS: track 5.98 -> 12.3 mm
- net 5V: track 100.9 -> 102.6 mm
Other:
- board text added: "Keyboard this way"

Commit message: Add files via upload
Parts:
- added R12: 1k, Resistor_THT:R_Axial_DIN0204_L3.6mm_D1.6mm_P5.08mm_Horizontal, F.Cu at (130.1, 95.8)
Routing:
- net 3.3V: track 0.00 -> 12.4 mm
- net GND: vias 36 -> 42
